File: kicad/ws_IT/IC555Demo/IC555Demo.kicad_pcb (KiCad board)
At the start: 2 copper layers, 33 x 32.4 mm, 8 parts, among them J1 CON02, U1 555

Commit message: Add JLC2KiCadLib
Other:
- board text added: "Woosong PCB"
- board text removed: "WooSong IT Pcb Trial v0.1.0"
- board text removed: "Woosong eventia PCB"
Changed lines of the file:
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@@
       (outputformat 1)
       (mirror false)
-      (drillshape 1)
+      (drillshape 0)
       (scaleselection 1)
-      (outputdirectory "")
+      (outputdirectory "gerber/")
     )
   )
@@
       (effects (font (size 1 1) (thickness 0.15)))
     )
+    (fp_text user "https://www.eleparts.co.kr/goods/view?no=9048" (at 0 0 unlocked) (layer "F.Fab")
+      (effects (font (size 1 1) (thickness 0.15)))
+    )
     (fp_text user "${REFERENCE}" (at 2.5 2.5 unlocked) (layer "F.Fab")
       (effects (font (size 1 1) (thickness 0.15)))
@@
     (effects (font (size 1.5 1.5) (thickness 0.3)))
   )
-  (gr_text "WooSong IT Pcb Trial v0.1.0" (at 159.385 57.785) (layer "B.Cu")
-    (effects (font (size 1.5 1.5) (thickness 0.3)) (justify mirror))
-  )
-  (gr_text "Woosong eventia PCB" (at 167.005 60.96) (layer "F.SilkS")
+  (gr_text "Woosong \nPCB" (at 169.545 61.595) (layer "F.SilkS")
     (effects (font (size 1 1) (thickness 0.15)))
   )
